File: PCB/Keyboard.kicad_pcb (KiCad board)
At the start: 2 copper layers, 109 x 68.5 mm, 43 parts, among them J1 USB_C_Receptacle_USB2.0_16P, SW1 SW_Push, SW10 SW_Push, SW11 SW_Push, SW2 RotaryEncoder_Switch, SW3 SW_Push, SW4 SW_Push, SW5 SW_Push, SW6 SW_Push, SW7 SW_Push, SW8 SW_Push, SW9 SW_Push, U1 STM32F072C8Tx, U2 USB6B1, U3 AMS1117-3.3

Commit message: Minor PCB changes
Parts:
- moved R1 10.8 mm to (120.6, 70.0), turned to 180 degrees
- moved H2 7.50 mm to (125.0, 30.0)
- moved H3 7.25 mm to (125.0, 87.5)
- moved C3 6.80 mm to (97.8, 33.2)
- moved SW1 5.83 mm to (121.8, 62.2)
- moved C9 5.46 mm to (114.8, 68.2), turned to 90 degrees
- moved C1 4.01 mm to (109.0, 83.8)
- moved C10 4.01 mm to (118.5, 82.2)
- moved C11 4.01 mm to (104.8, 88.8)
- moved C2 4.01 mm to (102.4, 31.7)
- moved C4 4.01 mm to (113.5, 82.3)
- moved C5 4.01 mm to (115.2, 71.5)
- moved C6 4.01 mm to (99.5, 72.5)
- moved C7 4.01 mm to (117.8, 77.5)
- moved C8 4.01 mm to (104.8, 84.0)
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Routing:
- net GND: track 5.67 -> 34.3 mm
- net +3.3V: track 153.2 -> 147.6 mm
- net /KR3: track 67.9 -> 63.8 mm
- net /KC2: track 86.1 -> 82.1 mm
- net /KC1: track 110.3 -> 106.4 mm
- net /KC3: track 57.9 -> 54.8 mm
- net /KR1: track 90.8 -> 89.2 mm
- net /BOOT0: track 27.1 -> 28.0 mm
- net /KR2: track 73.9 -> 73.3 mm
Other:
- board size 109 x 68.5 mm -> 100 x 68.5 mm
